File: Hardware/Electronics/boards/RADR PCB/RADR.kicad_pcb (KiCad board)
At the start: 4 copper layers, 109.8 x 50 mm, 98 parts, among them J1 SCREEN, J2 QWIIC, J3 ESP_IO0, J4 USB_C_Receptacle_USB2.0_16P, J5 BATT, J6 3.3V_INTERNAL, J7 GND, J8 ESP_EN, M1 Motor_DC, Q1 AO3400A, Q2 AO3400A, Q3 AO3400A, Q5 BC817, Q6 BC817, Q7 SI2301L, SW1 ENC_L, SW10 US_R, SW11 SW_DIP_x01, SW12 SW_DIP_x01, SW13 RESET, SW15 POWERSW, SW2 ENC_R, SW3 LS_1, SW4 LS_2, SW5 RS_1, SW6 RS_2, SW7 US_L, SW8 US_M_1, SW9 US_M_2, U1 ESP32-S3-WROOM-1, U10 ME6211C33M5, U2 AT24CS04-SSHM, U3 LSM6DS3, U4 CP2102-GMR, U6 MAX17048G+T10, U7 TP4054, U8 ME6211C33M5, U9 ME6211C33M5

Commit message: fabrication files for 0.4
Parts:
- D10, D8, D9: value XL-1010RGBC-WS2812B -> RGBC
- D5: value TJ-S1706SW6TGLC2G-A5 -> GRN
- D6: value TJ-S1706SW6TGLC6B-A5 -> BLU
- J4: value USB_C_Receptacle_USB2.0_16P -> USB_C_16P
- M1: value Motor_DC -> VIBRO
Changed lines of the file:
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@@
 	(layers
 		(0 "F.Cu" signal "Top Layer")
-		(4 "In1.Cu" power "3v3 - all domains")
-		(6 "In2.Cu" power "GND")
+		(4 "In1.Cu" power "In1")
+		(6 "In2.Cu" power "In2")
 		(2 "B.Cu" signal "Bottom Layer")
 		(9 "F.Adhes" user "F.Adhesive")
@@
 		(capping no)
 		(filling no)
+		(zone_defaults)
 		(aux_axis_origin 32.70107 185.822235)
 		(grid_origin 153.50107 129.272235)
@@
 			(outputformat 1)
 			(mirror no)
-			(drillshape 1)
+			(drillshape 0)
 			(scaleselection 1)
-			(outputdirectory "")
+			(outputdirectory "V0.4/")
 		)
 	)
@@
 			)
 		)
-		(property "Value" "XL-1010RGBC-WS2812B"
+		(property "Value" "RGBC"
 			(at 0 1.475 180)
 			(unlocked yes)
@@
 			)
 		)
+		(attr exclude_from_bom)
 		(duplicate_pad_numbers_are_jumpers no)
 		(fp_line
@@
 			)
 		)
-		(property "Value" "USB_C_Receptacle_USB2.0_16P"
+		(property "Value" "USB_C_16P"
 			(at 0 5.1 0)
 			(layer "F.Fab")
@@
 			)
 		)
-		(property "Value" "XL-1010RGBC-WS2812B"
+		(property "Value" "RGBC"
 			(at 0 1.475 0)
 			(unlocked yes)
@@
 			)
 		)
+		(attr exclude_from_bom)
 		(duplicate_pad_numbers_are_jumpers no)
 		(fp_circle
@@
 			)
 		)
+		(attr exclude_from_bom)
 		(duplicate_pad_numbers_are_jumpers no)
 		(fp_circle
@@
 			)
 		)
+		(attr exclude_from_bom)
 		(duplicate_pad_numbers_are_jumpers no)
 		(fp_line
@@
 			)
 		)
-		(property "Value" "XL-1010RGBC-WS2812B"
+		(property "Value" "RGBC"
 			(at 0 1.475 0)
 			(unlocked yes)
@@
 			)
 		)
-		(property "Value" "TJ-S1706SW6TGLC2G-A5"
+		(property "Value" "GRN"
 			(at 0 -1.43 180)
 			(layer "B.Fab")
@@
 			)
 		)
-		(property "Value" "TJ-S1706SW6TGLC6B-A5"
+		(property "Value" "BLU"
 			(at 0 -1.43 0)
 			(layer "B.Fab")
@@
 			)
 		)
-		(property "Value" "Motor_DC"
+		(property "Value" "VIBRO"
 			(at 0 -6.6 90)
 			(layer "B.Fab")
