File: Hardware/Electronics/boards/RADR PCB/RADR.kicad_sch (KiCad schematic)
At the start: 76 parts, among them J1 SCREEN, J2 QWIIC, J3 ESP_IO0, J8 ESP_EN, M1 Motor_DC, Q1 AO3400A, Q2 AO3400A, Q3 AO3400A, Q5 BC817, Q6 BC817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

Commit message: fabrication files for 0.4
Parts:
- BZ1: MFG (none) -> FUET; MPN (none) -> FUET-4020; lcsc-bom-key (none) -> C391027
- C10, C26, C35, C6, C8: MFG (none) -> Samsung Electro-Mechanics; MPN (none) -> CL05A105KA5NQNC; lcsc-bom-key (none) -> C52923
- C11, C15, C16, C17, C9: MFG (none) -> Samsung Electro-Mechanics; MPN (none) -> CL05A104KA5NNNC; lcsc-bom-key (none) -> C100072
- C28, C29, C30, C32, C33: MFG (none) -> Samsung Electro-Mechanics; MPN (none) -> CL31A107MQHNNNE; lcsc-bom-key (none) -> C15008
- C34: MFG (none) -> CL05B103KB5NNNC; MPN (none) -> CL05B103KB5NNNC; lcsc-bom-key (none) -> C15195
- D1, D2: MFG (none) -> HXY MOSFET; MPN (none) -> B5819W; lcsc-bom-key (none) -> C5345968
- D10, D8, D9: value XL-1010RGBC-WS2812B -> RGBC; MFG (none) -> XINGLIGHT; MPN (none) -> XL-1010RGBC-2812B; lcsc-bom-key (none) -> C5349953
- D5: value TJ-S1706SW6TGLC2G-A5 -> GRN; Characteristics (none) -> Green; MFG (none) -> TOGIALED; MPN (none) -> TJ-S1706SW6TGLC2G-A5; lcsc-bom-key (none) -> C273616
- D6: value TJ-S1706SW6TGLC6B-A5 -> BLU; Characteristics (none) -> Blue; MFG (none) -> TOGIALED; MPN (none) -> TJ-S1706SW6TGLC6B-A5; lcsc-bom-key (none) -> C273617
- J1: MFG (none) -> JUSHUO; MPN (none) -> AFC01-S14FCA-00; lcsc-bom-key (none) -> C262663
- J2: MFG (none) -> JST; MPN (none) -> SM04B-SRSS-TB(LF)(SN); lcsc-bom-key (none) -> C160404
- J3, J8: now left out of the parts list
- M1: value Motor_DC -> VIBRO; MFG (none) -> KOTL; MPN (none) -> Z3OC1T8219731; lcsc-bom-key (none) -> C2894731
- Q1, Q2, Q3: MFG (none) -> AOS; MPN (none) -> AO3400A; lcsc-bom-key (none) -> C20917
- Q5, Q6: MFG (none) -> Nexperia; MPN (none) -> BC817-25,215; lcsc-bom-key (none) -> C39828
- R1: MFG (none) -> YAGEO; MPN (none) -> RC0603JR-0710RL; lcsc-bom-key (none) -> C109317
- R10, R9: MFG (none) -> YAGEO; MPN (none) -> RC0402FR-07100RL; lcsc-bom-key (none) -> C106232
- R11: MFG (none) -> YAGEO; MPN (none) -> RC0402FR-071KL; lcsc-bom-key (none) -> C106235
- R19: MFG (none) -> YAGEO; MPN (none) -> RC0402FR-07330RL; lcsc-bom-key (none) -> C105875
- R22, R23, R24, R25, R26, R32, R35, R36, R7, R8: MFG (none) -> YAGEO; MPN (none) -> RC0402FR-0710KL; lcsc-bom-key (none) -> C60490
- R34: MFG (none) -> YAGEO; MPN (none) -> RC0402FR-075K1L; lcsc-bom-key (none) -> C105872
- R40, R41: MFG (none) -> YAGEO; MPN (none) -> RC0402FR-074K7L; lcsc-bom-key (none) -> C105871
- SW1, SW2: MFG (none) -> ALPSALPINE; MPN (none) -> EC12E24204A8; lcsc-bom-key (none) -> C470598
- SW10, SW7, SW8, SW9: MFG (none) -> HCTL; MPN (none) -> TC-6610-9-260G; lcsc-bom-key (none) -> C2845257
- SW11, SW12: MFG (none) -> SHOU HAN; MPN (none) -> 2.54-1P TPGT; lcsc-bom-key (none) -> C7421519
- SW13, SW3, SW4, SW5, SW6: MFG (none) -> SHOU HAN; MPN (none) -> TS24CA; lcsc-bom-key (none) -> C393942
- U1: Characteristics (none) -> N16R8; MFG (none) -> ESPRESSIF; MPN (none) -> C2913202 ESP32-S3-WROOM-1-N16R8 ESPRESSIF N16R8; lcsc-bom-key (none) -> C2913202
- U2: MFG (none) -> MICROCHIP; MPN (none) -> AT24C04C-SSHM-T; lcsc-bom-key (none) -> C6205
- U3: MFG (none) -> ST; MPN (none) -> LSM6DS3TR; lcsc-bom-key (none) -> C95230
- U4: MFG (none) -> SILICON LABS; MPN (none) -> CP2102-GMR; lcsc-bom-key (none) -> C6568
Other:
- company: (none) -> Research and Desire
- title: (none) -> RADR - OSSM Wireless Remote
