File: Hardware/Electronics/boards/RADR PCB/power.kicad_sch (KiCad schematic)
At the start: 25 parts, among them J4 USB_C_Receptacle_USB2.0_16P, J5 BATT, J6 3.3V_INTERNAL, J7 GND, Q7 SI2301L, SW15 POWERSW, U10 ME6211C33M5, U6 MAX17048G+T10, U7 TP4054, U8 ME6211C33M5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

Commit message: fabrication files for 0.4
Parts:
- C14, C23, C24, C25, C27: MFG (none) -> Samsung Electro-Mechanics; MPN (none) -> CL05A105KA5NQNC; lcsc-bom-key (none) -> C52923
- C18, C19, C20: MFG (none) -> Samsung Electro-Mechanics; MPN (none) -> CL05A225KO5NQNC; lcsc-bom-key (none) -> C170151
- D3: MFG (none) -> HXY MOSFET; MPN (none) -> B5819W; lcsc-bom-key (none) -> C5345968
- J4: value USB_C_Receptacle_USB2.0_16P -> USB_C_16P; MFG (none) -> Korean Hroparts Elec; MPN (none) -> TYPE-C-31-M-12; lcsc-bom-key (none) -> C165948
- J5: MFG (none) -> JST; MPN (none) -> S2B-PH-K(LF)(SN); lcsc-bom-key (none) -> C265016
- J6, J7: now left out of the parts list
- Q7: MFG (none) -> TWGMC; MPN (none) -> SI2301; lcsc-bom-key (none) -> C727151
- R16: MFG (none) -> YAGEO; MPN (none) -> RC0402FR-071KL; lcsc-bom-key (none) -> C106235
- R18: MFG (none) -> YAGEO; MPN (none) -> RC0402FR-072KL; lcsc-bom-key (none) -> C60488
- R20, R21: MFG (none) -> YAGEO; MPN (none) -> RC0402FR-075K1L; lcsc-bom-key (none) -> C105872
- R39: MFG (none) -> YAGEO; MPN (none) -> RC0402FR-0710KL; lcsc-bom-key (none) -> C60490
- SW15: MFG (none) -> SHOU HAN; MPN (none) -> SK12D07VG5; lcsc-bom-key (none) -> C431548
- U10, U8, U9: MFG (none) -> MICRONE; MPN (none) -> ME6211C33R5G; lcsc-bom-key (none) -> C235316
- U6: MFG (none) -> MAXIM; MPN (none) -> MAX17048G+T10; lcsc-bom-key (none) -> C2682616
- U7: MFG (none) -> JSMSEMI; MPN (none) -> TP4054; lcsc-bom-key (none) -> C5381776
Other:
- company: (none) -> Research and Desire
- title: (none) -> RADR - OSSM Wireless Remote
